File: 4Keys.kicad_pcb (KiCad board)
At the start: 2 copper layers, 29 parts, among them J1 OLED1, J2 OLED2, SW1 SW_Reset, U1 ATmega32U4-AU, Y1 16MHz

Commit message: Update PCB
Parts:
- C5: value C_Small -> 1uF
- D2, F1, R1, R2, R4, R5: moved to F.Cu
- moved F1 72.1 mm to (177.5, 35.4), turned to 90 degrees
- moved R4 68.9 mm to (185.6, 37.0), turned to 90 degrees
- moved R5 68.6 mm to (183.0, 37.1), turned to 270 degrees
- moved Y1 61.5 mm to (186.5, 55.9), turned to 90 degrees
- moved D1 59.7 mm to (194.1, 36.8)
- moved C7 57.3 mm to (197.1, 44.0), turned to 180 degrees
- moved D2 56.2 mm to (193.7, 44.5), turned to 90 degrees
- moved C2 54.4 mm to (186.5, 52.4), turned to 180 degrees
- moved C1 52.5 mm to (186.5, 59.4)
- moved C6 50.9 mm to (197.1, 64.0)
- moved R6 50.1 mm to (202.9, 44.0), turned to 180 degrees
- moved R2 49.0 mm to (201.0, 52.1), turned to 90 degrees
- moved R3 48.1 mm to (196.0, 68.1), turned to 90 degrees
- moved C4 44.7 mm to (210.0, 50.1), turned to 270 degrees
- moved R1 43.6 mm to (204.0, 52.0), turned to 90 degrees
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Connections:
- D4 pad 1: row0 -> row1
- MXDn1 pad 1: col0 -> col1
- MXLeft1 pad 1: col1 -> col0
- MXRight1 pad 1: col1 -> col2
- MXUp1 pad 1: col0 -> col1
- U1 pad 11: Net-(U1-Pad11) -> col2
Routing:
- net +5V: track 0.00 -> 56.5 mm
- net VCC: track 0.00 -> 37.2 mm
- net D+: track 0.00 -> 20.5 mm
- net GND: track 0.00 -> 19.7 mm
- net D-: track 0.00 -> 11.8 mm, vias 0 -> 2
- net Net-(R5-Pad2): track 0.00 -> 5.65 mm
- net Net-(R6-Pad2): track 0.00 -> 4.85 mm
- net Net-(R4-Pad2): track 0.00 -> 4.07 mm
Other:
- board outline added: 103.2 x 52.4 mm
- net class Default: trace_width 0.25 -> 0.254
- net class power added: clearance 0.2, trace_width 0.381, via_dia 0.8, via_drill 0.4
