File: _autosave-4Keys.kicad_pcb (KiCad board)
At the start: 2 copper layers, 103.2 x 52.4 mm, 29 parts, among them J1 OLED1, J2 OLED2, SW1 SW_Reset, U1 ATmega32U4-AU, Y1 16MHz

Commit message: update pcb
Routing:
- net SCL: track 88.3 -> 99.3 mm, vias 0 -> 1
- net SDA: track 89.0 -> 99.7 mm, vias 0 -> 1
Changed lines of the file:
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@@
     (thickness 1.6)
     (drawings 8)
-    (tracks 222)
+    (tracks 233)
     (zones 0)
     (modules 29)
@@
   (segment (start 230.279 77.3) (end 231.79 75.789) (width 0.254) (layer B.Cu) (net 15))
   (segment (start 148.6585 77.3) (end 230.279 77.3) (width 0.254) (layer B.Cu) (net 15))
+  (segment (start 196.12275 52.38125) (end 198.8595 55.118) (width 0.254) (layer B.Cu) (net 15))
+  (segment (start 195.11875 52.38125) (end 196.12275 52.38125) (width 0.254) (layer B.Cu) (net 15))
+  (segment (start 198.8595 55.118) (end 204.724 55.118) (width 0.254) (layer B.Cu) (net 15))
+  (via (at 204.727 55.372) (size 0.8) (drill 0.4) (layers F.Cu B.Cu) (net 15))
+  (segment (start 204.724 55.118) (end 204.724 55.369) (width 0.254) (layer B.Cu) (net 15))
+  (segment (start 204.724 55.369) (end 204.727 55.372) (width 0.254) (layer B.Cu) (net 15))
   (segment (start 229.29 75.789) (end 227.079 78) (width 0.254) (layer F.Cu) (net 16))
   (segment (start 229.29 74.56) (end 229.29 75.789) (width 0.254) (layer F.Cu) (net 16))
@@
   (segment (start 227.079 78) (end 146.8585 78) (width 0.254) (layer F.Cu) (net 16))
   (segment (start 229.29 74.56) (end 229.29 74.46) (width 0.254) (layer F.Cu) (net 16))
+  (segment (start 196.12275 51.58125) (end 198.8975 54.356) (width 0.254) (layer B.Cu) (net 16))
+  (segment (start 195.11875 51.58125) (end 196.12275 51.58125) (width 0.254) (layer B.Cu) (net 16))
+  (segment (start 198.8975 54.356) (end 204.724 54.356) (width 0.254) (layer B.Cu) (net 16))
+  (via (at 204.727 54.356) (size 0.8) (drill 0.4) (layers F.Cu B.Cu) (net 16))
+  (segment (start 204.724 54.356) (end 204.727 54.356) (width 0.254) (layer B.Cu) (net 16))
   (segment (start 162.8775 64.419788) (end 176.697288 50.6) (width 0.254) (layer F.Cu) (net 17))
   (segment (start 162.8775 64.92875) (end 162.8775 64.419788) (width 0.254) (layer F.Cu) (net 17))
